Commit message: default colors

File: src/my_car/description/robot_core.xacro (robot description, xacro)
@@ -1,3 +1,15 @@
 <?xml version="1.0"?>
 <robot xmlns:xacro="http://www.ros.org/wiki/xacro">
+    <material name="white">
+        <color rgba="1 1 1 1"/>
+    </material>
+    <material name="black">
+        <color rgba="0 0 0 1"/>
+    </material>
+    <material name="orange">
+        <color rgba="1 0.5 0.1 1"/>
+    </material>
+    <material name="blue">
+        <color rgba="0.2 0.2 1 1"/>
+    </material>
 </robot>

Commit message: base link is the center of the two drive wheels

File: src/my_car/description/robot_core.xacro (robot description, xacro)
@@ -13,3 +13,5 @@
         <color rgba="0.2 0.2 1 1"/>
     </material>
+    <link name="base_link">
+    </link>
 </robot>

Commit message: made the chasis and launcehed rviz2

File: src/my_car/description/robot_core.xacro (robot description, xacro)
@@ -8,5 +8,5 @@
     </material>
     <material name="orange">
-        <color rgba="1 0.5 0.1 1"/>
+        <color rgba="1 0.3 0.1 1"/>
     </material>
     <material name="blue">
@@ -15,3 +15,17 @@
     <link name="base_link">
     </link>
+    <joint name="chassis_joint" type="fixed">
+        <parent link="base_link"/>
+        <child link="chassis"/>
+        <origin xyz="-0.1 0 0"/>
+    </joint>
+    <link name="chassis">
+        <visual>
+            <origin xyz="0.15 0 0.075"/>
+            <geometry>
+                <box size="0.3 0.3 0.15"/>
+            </geometry>
+            <material name="white"/>
+        </visual>
+    </link>
 </robot>

Commit message: the wheels are there but they long

File: src/my_car/description/robot_core.xacro (robot description, xacro)
@@ -32,3 +32,32 @@
     </link>
     <!-- Left Wheel link-->
+    <joint name="left_wheel_joint" type="continuous">
+        <parent link="base_link"/>
+        <child link="left_wheel"/>
+        <origin xyz="0 0.175 0" rpy="-${pi/2} 0 0"/>
+        <axis xyz="0 0 1"/>
+    </joint>
+    <link name="left_wheel">
+        <visual>
+            <geometry>
+                <cylinder radius="0.05" length="0.4"/>
+            </geometry>
+            <material name="blue"/>
+        </visual>
+    </link>
+    <!-- right Wheel link-->
+    <joint name="right_wheel_joint" type="continuous">
+        <parent link="base_link"/>
+        <child link="right_wheel"/>
+        <origin xyz="0 -0.175 0" rpy="${pi/2} 0 0"/>
+        <axis xyz="0 0 1"/>
+    </joint>
+    <link name="right_wheel">
+        <visual>
+            <geometry>
+                <cylinder radius="0.05" length="0.4"/>
+            </geometry>
+            <material name="blue"/>
+        </visual>
+    </link>
 </robot>

Commit message: changed the length of the wheels to something reasonable

File: src/my_car/description/robot_core.xacro (robot description, xacro)
@@ -41,5 +41,5 @@
         <visual>
             <geometry>
-                <cylinder radius="0.05" length="0.4"/>
+                <cylinder radius="0.05" length="0.04"/>
             </geometry>
             <material name="blue"/>
@@ -56,5 +56,5 @@
         <visual>
             <geometry>
-                <cylinder radius="0.05" length="0.4"/>
+                <cylinder radius="0.05" length="0.04"/>
             </geometry>
             <material name="blue"/>

Commit message: the right wheel should go forward when i turn forwards

File: src/my_car/description/robot_core.xacro (robot description, xacro)
@@ -51,5 +51,5 @@
         <child link="right_wheel"/>
         <origin xyz="0 -0.175 0" rpy="${pi/2} 0 0"/>
-        <axis xyz="0 0 1"/>
+        <axis xyz="0 0 -1"/>
     </joint>
     <link name="right_wheel">

Commit message: the caster wheen done

File: src/my_car/description/robot_core.xacro (robot description, xacro)
@@ -61,3 +61,17 @@
         </visual>
     </link>
+    <!-- Caster Wheel link-->
+    <joint name="caster_wheel_joint" type="fixed">
+        <parent link="chassis"/>
+        <child link="caster_wheel"/>
+        <origin xyz="0.24 0 0"/>
+    </joint>
+    <link name="caster_wheel">
+        <visual>
+            <geometry>
+                <sphere radius="0.05"/>
+            </geometry>
+            <material name="black"/>
+        </visual>
+    </link>
 </robot>

Commit message: collision added only left with enertia

File: src/my_car/description/robot_core.xacro (robot description, xacro)
@@ -30,4 +30,10 @@
             <material name="white"/>
         </visual>
+        <collision>
+            <origin xyz="0.15 0 0.075"/>
+            <geometry>
+                <box size="0.3 0.3 0.15"/>
+            </geometry>
+        </collision>
     </link>
     <!-- Left Wheel link-->
@@ -45,4 +51,9 @@
             <material name="blue"/>
         </visual>
+        <collision>
+            <geometry>
+                <cylinder radius="0.05" length="0.04"/>
+            </geometry>
+        </collision>
     </link>
     <!-- right Wheel link-->
@@ -60,4 +71,9 @@
             <material name="blue"/>
         </visual>
+        <collision>
+            <geometry>
+                <cylinder radius="0.05" length="0.04"/>
+            </geometry>
+        </collision>
     </link>
     <!-- Caster Wheel link-->
@@ -74,4 +90,9 @@
             <material name="black"/>
         </visual>
+        <collision>
+            <geometry>
+                <sphere radius="0.05"/>
+            </geometry>
+        </collision>
     </link>
 </robot>

Commit message: added inertia

File: src/my_car/description/robot_core.xacro (robot description, xacro)
@@ -38,4 +38,7 @@
             </geometry>
         </collision>
+        <xacro:inertial_box mass="1.0" x="0.3" y="0.3" z="0.15">
+            <origin xyz="0.15 0 0.075" rpy="0 0 0"/>
+        </xacro:inertial_box>
     </link>
     <!-- Left Wheel link-->
@@ -58,4 +61,7 @@
             </geometry>
         </collision>
+        <xacro:inertial_cylinder mass="0.1" length="0.04" radius="0.05">
+            <origin xyz="0 0 0" rpy="0 0 0"/>
+        </xacro:inertial_cylinder>
     </link>
     <!-- right Wheel link-->
@@ -78,4 +84,7 @@
             </geometry>
         </collision>
+        <xacro:inertial_cylinder mass="0.1" length="0.04" radius="0.05">
+            <origin xyz="0 0 0" rpy="0 0 0"/>
+        </xacro:inertial_cylinder>
     </link>
     <!-- Caster Wheel link-->
@@ -97,4 +106,7 @@
             </geometry>
         </collision>
+        <xacro:inertial_sphere mass="0.1" radius="0.05">
+            <origin xyz="0 0 0" rpy="0 0 0"/>
+        </xacro:inertial_sphere>
     </link>
 </robot>
